Commit message: first spot mini

File: mark_I/assets2/spotmini.urdf (robot description, URDF)
Before this commit: robot rex_full, 23 links, 22 joints
Links:
- link base_link: mass 1.20 -> 2.80
- link chassis_front_link: mass 0.05 -> 0.20
- link chassis_rear_link: mass 0.05 -> 0.20
- link front_left_foot_link: geometry collision box size=0.026 0.020 0.115; visual mesh filename=stl/lfoot.stl scale=0.001 0.001 0.001
- link front_left_leg_link: mass 0.1 -> 0.15; geometry collision box size=0.028 0.036 0.12; visual mesh filename=stl/larm.stl scale=0.001 0.001 0.001
- link front_left_leg_link_cover: mass 0.5 -> None; geometry visual mesh filename=stl/larm_cover.stl scale=0.001 0.001 0.001
- link front_left_toe_link: mass 0.005 -> 0.05; geometry collision sphere radius=0.02; visual mesh filename=stl/foot.stl scale=0.001 0.001 0.001
- link front_right_foot_link: geometry collision box size=0.026 0.020 0.115; visual mesh filename=stl/rfoot.stl scale=0.001 0.001 0.001
- link front_right_leg_link: mass 0.1 -> 0.15; geometry collision box size=0.028 0.036 0.12; visual mesh filename=stl/rarm.stl scale=0.001 0.001 0.001
- link front_right_leg_link_cover: mass 0.5 -> None; geometry visual mesh filename=stl/rarm_cover.stl scale=0.001 0.001 0.001
- link front_right_toe_link: mass 0.005 -> 0.05; geometry collision sphere radius=0.02; visual mesh filename=stl/foot.stl scale=0.001 0.001 0.001
- link rear_left_foot_link: geometry collision box size=0.026 0.020 0.115; visual mesh filename=stl/lfoot.stl scale=0.001 0.001 0.001
- link rear_left_leg_link: mass 0.10 -> 0.15; geometry collision box size=0.028 0.036 0.12; visual mesh filename=stl/larm.stl scale=0.001 0.001 0.001
- link rear_left_leg_link_cover: mass 0.5 -> None; geometry visual mesh filename=stl/larm_cover.stl scale=0.001 0.001 0.001
- link rear_left_toe_link: mass 0.005 -> 0.05; geometry collision sphere radius=0.02; visual mesh filename=stl/foot.stl scale=0.001 0.001 0.001
- link rear_right_foot_link: geometry collision box size=0.026 0.020 0.115; visual mesh filename=stl/rfoot.stl scale=0.001 0.001 0.001
- link rear_right_leg_link: mass 0.10 -> 0.15; geometry collision box size=0.028 0.036 0.12; visual mesh filename=stl/rarm.stl scale=0.001 0.001 0.001
- link rear_right_leg_link_cover: mass 0.5 -> None; geometry visual mesh filename=stl/rarm_cover.stl scale=0.001 0.001 0.001
- link rear_right_toe_link: mass 0.005 -> 0.05; geometry collision sphere radius=0.02; visual mesh filename=stl/foot.stl scale=0.001 0.001 0.001
Joints:
- joint chassis_base_front: child chassis_front_link -> front_link
- joint chassis_base_rear: child chassis_rear_link -> rear_link
- joint foot_motor_FL: limit lower=-3.14 upper=3.14 effort=100.0 velocity=0.5 -> lower=-0.1 upper=2.59 effort=1000.0 velocity=0.5; origin xyz=0.002 -0.02 -0.16 rpy=0 0 0 -> xyz=-0.01 0 -0.12 rpy=0 0 0
- joint foot_motor_FR: limit lower=-3.14 upper=3.14 effort=100.0 velocity=0.5 -> lower=-0.1 upper=2.59 effort=1000.0 velocity=0.5; origin xyz=0.002 0.02 -0.16 rpy=0 0 0 -> xyz=-0.01 0 -0.12 rpy=0 0 0
- joint foot_motor_RL: limit lower=-3.14 upper=3.14 effort=100.0 velocity=0.5 -> lower=-0.1 upper=2.59 effort=1000.0 velocity=0.5; origin xyz=0.002 -0.02 -0.16 rpy=0 0 0 -> xyz=-0.01 0 -0.12 rpy=0 0 0
- joint foot_motor_RR: limit lower=-3.14 upper=3.14 effort=100.0 velocity=0.5 -> lower=-0.1 upper=2.59 effort=1000.0 velocity=0.5; origin xyz=0.002 0.02 -0.16 rpy=0 0 0 -> xyz=-0.01 0 -0.12 rpy=0 0 0
- joint motor_leg_FL: limit lower=-1.57 upper=1.57 effort=100.0 velocity=0.5 -> lower=-2.666 upper=1.548 effort=1000.0 velocity=0.5
- joint motor_leg_FR: limit lower=-1.57 upper=1.57 effort=100.0 velocity=0.5 -> lower=-2.666 upper=1.548 effort=1000.0 velocity=0.5; origin xyz=0 0.042 0 rpy=0 0 0 -> xyz=0 0.052 0 rpy=0 0 0
- joint motor_leg_RL: limit lower=-1.57 upper=1.57 effort=100.0 velocity=0.5 -> lower=-2.666 upper=1.548 effort=1000.0 velocity=0.5
- joint motor_leg_RR: limit lower=-1.57 upper=1.57 effort=100.0 velocity=0.5 -> lower=-2.666 upper=1.548 effort=1000.0 velocity=0.5; origin xyz=0 0.042 0 rpy=0 0 0 -> xyz=0 0.052 0 rpy=0 0 0
- joint motor_shoulder_FL: limit lower=-1.0 upper=1.0 effort=100.0 velocity=0.7 -> lower=-0.548 upper=0.548 effort=1000.0 velocity=0.7
- joint motor_shoulder_FR: limit lower=-1.0 upper=1.0 effort=100.0 velocity=0.7 -> lower=-0.548 upper=0.548 effort=1000.0 velocity=0.7
- joint motor_shoulder_RL: limit lower=-1.0 upper=1.0 effort=100.0 velocity=0.7 -> lower=-0.548 upper=0.548 effort=1000.0 velocity=0.7
- joint motor_shoulder_RR: limit lower=-1.0 upper=1.0 effort=100.0 velocity=0.7 -> lower=-0.548 upper=0.548 effort=1000.0 velocity=0.7
